File: src/IM920sL_module.brd (EAGLE design)
At the start: 160 x 100 mm, 11 parts, among them CN1 20P5.0-JMCS-G-TF(N), SW1 一般的なタクトスイッチ, SW2 一般的なタクトスイッチ

Commit message: Eagle移行前_配線図完成
Parts:
- removed LED1: SML-E12V8WT86, SML-E12V8WT86:SML-E12V8WT86
- added LED: SML-E12V8WT86, SML-E12V8WT86:SML-E12V8WT86
- moved AD_MODE 67.9 mm to (32.1, 27.5)
- moved R2 58.2 mm to (14.1, 12.9), flipped to the bottom
- moved R3 58.2 mm to (14.1, 10.4), flipped to the bottom
- moved SW2 56.2 mm to (32.3, 9.56), turned to 270 degrees
- moved C1 55.6 mm to (17.1, 4.70), turned to 90 degrees
- moved SW1 53.8 mm to (32.3, 19.5), turned to 270 degrees
- moved JP2 43.3 mm to (40.7, 15.4), turned to 270 degrees
- moved R1 33.7 mm to (22.8, 3.32), turned to 180 degrees
- moved JP1 27.1 mm to (2.62, 15.4), turned to 270 degrees
- moved CN1 12.0 mm to (12.4, 4.50)
Connections:
- net GND: now also LED.K; no longer LED1.K, SW1.T1, SW2.T1
- net N$1: now also LED.A; no longer LED1.A
- net REG: no longer SW1.T3
- net RESET: no longer SW2.T3
Routing:
- net P8: track 0.00 -> 48.8 mm
- net P2: track 0.00 -> 42.4 mm
- net REG: track 0.00 -> 42.3 mm
- net P10: track 0.00 -> 40.1 mm, vias 0 -> 1
- net P4: track 0.00 -> 39.6 mm
- net P6: track 0.00 -> 36.8 mm
- net RESET: track 0.00 -> 34.0 mm
- net P9: track 0.00 -> 29.4 mm, vias 0 -> 2
- net P1: track 0.00 -> 27.3 mm
- net STATUS: track 0.00 -> 27.2 mm
- net P3: track 0.00 -> 23.9 mm, vias 0 -> 1
- net P5: track 0.00 -> 22.0 mm, vias 0 -> 1
- net VCC: track 0.00 -> 20.9 mm
- net P7: track 0.00 -> 19.9 mm, vias 0 -> 1
- net N$1: track 0.00 -> 8.98 mm
- added copper zone on layer 1, net GND
- added copper zone on layer 16, net VCC
Other:
- board size 160 x 100 mm -> 43.6 x 31.9 mm
