File: src/IM920sL_module.sch (EAGLE design)
At the start: 11 parts, among them CN1 20P5.0-JMCS-G-TF(N), SW1 一般的なタクトスイッチ, SW2 一般的なタクトスイッチ

Commit message: Eagle移行前_配線図完成
Parts:
- renumbered LED1 to LED
