File: src/IM920sL_module(KiCad)/IM920sL_module.kicad_pcb (KiCad board)
At the start: 2 copper layers, 43.6 x 31.9 mm, 12 parts, among them CN1 20P5.0-JMCS-G-TF(N), SW1 一般的なタクトスイッチ, SW2 一般的なタクトスイッチ

Commit message: 基板デザインの改良
Routing:
- net /RESET: track 34.0 -> 34.7 mm
Other:
- board size 43.6 x 31.9 mm -> 43.6 x 31.8 mm
